File: hardware/Deck_Mainboard/Deck_Mainboard.kicad_pcb (KiCad board)
At the start: 2 copper layers, 98 x 62 mm, 60 parts, among them J2 BUTTONS, J3 ENCODERS, J4 LCD, J5 SD, J6 ADDITIONAL PINS, J7 DEBUG, J8 USB_C_Receptacle_USB2.0_16P, SW1 RESET, SW2 BOOTSEL, U1 RP2350B, U2 USBLC6-2SC6, U3 AP2112K-3.3, U4 APS6404L-3SQRx-SN, U5 W25Q128JVS, X1 ABM8-272-T3

Commit message: temporary commit for validation
Parts:
- C4: value 1u -> 10u
- moved SW1 29.2 mm to (96.8, 109.0), turned to -90 degrees
- moved R13 25.9 mm to (95.2, 102.2)
- moved SW2 24.9 mm to (114.5, 75.0), turned to -90 degrees
- moved J7 7.77 mm to (83.5, 110.5)
- moved D1 7.13 mm to (97.3, 75.4)
- moved R11 7.13 mm to (97.3, 78.7), turned to 90 degrees
- moved R12 1.58 mm to (115.8, 82.2), turned to 45 degrees
- moved C16 0.69 mm to (101.5, 89.7)
- moved J2 0.20 mm to (130.0, 119.0)
- moved R14 0.19 mm to (101.5, 93.2)
- moved C10 0.19 mm to (101.5, 94.2)
- moved C17 0.19 mm to (101.5, 91.8)
Connections:
- J2 pad 2: /SW1 -> /SW6
- J2 pad 3: /SW2 -> /SW5
- J2 pad 4: /SW3 -> /SW4
- J2 pad 5: /SW4 -> /SW3
- J2 pad 6: /SW5 -> /SW2
- J2 pad 7: /SW6 -> /SW1
Routing:
- net /SD_MISO: track 0.00 -> 86.9 mm
- net /SD_SCK: track 0.00 -> 84.0 mm
- net /SD_CS: track 0.00 -> 83.2 mm, vias 0 -> 2
- net /SD_MOSI: track 0.00 -> 79.9 mm, vias 0 -> 2
- net /ENC1_SW: track 0.00 -> 38.5 mm
- net /ENC2_A: track 0.00 -> 36.5 mm
- net /GPIO27: track 0.00 -> 36.3 mm, vias 0 -> 2
- net /CS: track 0.00 -> 36.2 mm
- net /RESET: track 0.00 -> 35.0 mm, vias 0 -> 2
- net /D/C: track 0.00 -> 34.9 mm
- net /GPIO26: track 0.00 -> 34.9 mm, vias 0 -> 2
- net /MOSI(SDI): track 0.00 -> 34.7 mm
- net /MISO(SDO): track 0.00 -> 34.7 mm
- net /ENC2_B: track 0.00 -> 34.6 mm
- net /SCLK: track 0.00 -> 34.5 mm
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