File: hardware/Deck_Mainboard/Deck_Mainboard.kicad_pcb (KiCad board)
At the start: 2 copper layers, 98 x 62 mm, 60 parts, among them J2 BUTTONS, J3 ENCODERS, J4 LCD, J5 SD, J6 ADDITIONAL PINS, J7 DEBUG, J8 USB_C_Receptacle_USB2.0_16P, SW1 RESET, SW2 BOOTSEL, U1 RP2350B, U2 USBLC6-2SC6, U3 AP2112K-3.3, U4 APS6404L-3SQRx-SN, U5 W25Q128JVS, X1 ABM8-272-T3

Commit message: hw: connectors routing
Parts:
- C4: value 1u -> 10u
- moved SW1 29.2 mm to (96.8, 109.0), turned to -90 degrees
- moved R13 25.9 mm to (95.2, 102.2)
- moved SW2 24.9 mm to (114.5, 75.0), turned to -90 degrees
- moved J7 7.77 mm to (83.5, 110.5)
- moved D1 7.13 mm to (97.3, 75.4)
- moved R11 7.13 mm to (97.3, 78.7), turned to 90 degrees
- moved R12 1.58 mm to (115.8, 82.2), turned to 45 degrees
- moved C16 0.69 mm to (101.5, 89.7)
- moved J2 0.20 mm to (130.0, 119.0)
- moved R14 0.19 mm to (101.5, 93.2)
- moved C10 0.19 mm to (101.5, 94.2)
- moved C17 0.19 mm to (101.5, 91.8)
Connections:
- J2 pad 2: /SW1 -> /SW6
- J2 pad 3: /SW2 -> /SW5
- J2 pad 4: /SW3 -> /SW4
- J2 pad 5: /SW4 -> /SW3
- J2 pad 6: /SW5 -> /SW2
- J2 pad 7: /SW6 -> /SW1
Routing:
- net /SD_MISO: track 0.00 -> 86.9 mm
- net /SD_SCK: track 0.00 -> 84.0 mm
- net /SD_CS: track 0.00 -> 83.2 mm, vias 0 -> 2
- net /SD_MOSI: track 0.00 -> 79.9 mm, vias 0 -> 2
- net /ENC1_SW: track 0.00 -> 38.6 mm
- net /ENC2_A: track 0.00 -> 36.5 mm
- net /CS: track 0.00 -> 36.4 mm
- net /GPIO27: track 0.00 -> 36.3 mm, vias 0 -> 2
- net /D/C: track 0.00 -> 35.1 mm
- net /RESET: track 0.00 -> 35.0 mm, vias 0 -> 2
- net /MOSI(SDI): track 0.00 -> 35.0 mm
- net /GPIO26: track 0.00 -> 34.9 mm, vias 0 -> 2
- net /SCLK: track 0.00 -> 34.9 mm
- net /LED: track 0.00 -> 34.8 mm
- net /MISO(SDO): track 0.00 -> 34.7 mm
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
Commit message: hw: pcbs complete
Parts:
- CR1: value MBR120VLSFT1G -> SDO_SOD-123FL_ONS
- H5, H6: value MH -> MH_P; footprint MountingHole:MountingHole_3.2mm_M3 -> MountingHole:MountingHole_3.2mm_M3_Pad
- J8: footprint deckLib:USB_C_4805 -> deckLib:USB_C_vertical
- X1: footprint Crystal:ABM8-272-T3_ABR -> deckLib:ABM8-272-T3_ABR
- moved H5 21.1 mm to (133.2, 79.6)
- moved H6 21.0 mm to (153.2, 79.6)
- moved R4 10.1 mm to (142.8, 75.3), turned to 90 degrees
- moved J7 7.38 mm to (86.9, 103.9)
- moved R5 4.93 mm to (145.6, 84.5)
- moved J8 2.19 mm to (143.2, 79.6), turned to 0 degrees
- moved R6 1.21 mm to (143.9, 97.9)
- moved U3 1.21 mm to (140.8, 98.3)
- moved SW1 1.19 mm to (97.5, 108.0)
- moved R13 1.19 mm to (95.8, 101.2)
- moved C4 0.69 mm to (142.5, 100.9)
- moved C5 0.69 mm to (140.2, 100.9)
- moved C15 0.50 mm to (109.2, 85.2)
- moved F1 0.50 mm to (148.2, 86.5)
- moved CR1 0.10 mm to (148.2, 93.0)
Connections:
- C4 pad 1: Net-(U3-VIN) -> +5V
- CR1 pad 1: Net-(U3-VIN) -> +5V
- CR1 pad 2: +5V -> /VBUS
- F1 pad 2: +5V -> /VBUS
- R6 pad 2: Net-(U3-VIN) -> +5V
- U2 pad 5: +5V -> /VBUS
- U3 pad 1: Net-(U3-VIN) -> +5V
Routing:
- net +5V: track 2.34 -> 151.1 mm, vias 0 -> 2
- net GND: track 5.43 -> 46.7 mm, vias 10 -> 46
- net +1.1V: track 8.85 -> 26.2 mm, vias 3 -> 9
- net +3.3V: track 27.7 -> 41.4 mm
- net /VBUS: track 0.00 -> 9.83 mm
- net Net-(U3-VIN): track 9.49 -> 0.00 mm
- net Net-(F1-Pad1): track 12.0 -> 19.6 mm, vias 0 -> 2
- net /SWDIO: track 24.5 -> 17.4 mm
- net /SWCLK: track 27.4 -> 21.4 mm
- net /USB_N: track 6.77 -> 11.4 mm, vias 0 -> 3
- net /USB_P: track 5.68 -> 7.39 mm
- net Net-(J8-CC1): track 3.79 -> 2.40 mm
- net /RUN: track 21.2 -> 19.9 mm
- added copper zone on F.Cu, net +1.1V
- added copper zone on F.Cu, net +3.3V
- added copper zone on B.Cu, net GND
Other:
- board size 98 x 62 mm -> 98 x 63.2 mm
- board text added: "+3.3V"
- board text added: "+5V"
- board text added: "1 A"
- board text added: "1 B"
- board text added: "1 SW"
- board text added: "2"
- board text added: "2 A"
- board text added: "2 B"
- board text added: "2 SW"
- board text added: "3 A"
- board text added: "3 B"
- board text added: "3 SW"
- board text added: "CS"
- board text added: "D/C"
- board text added: "GND"
- board text added: "GPIO23"
- board text added: "GPIO24"
- board text added: "GPIO26"
- board text added: "GPIO27"
- board text added: "LED"
- board text added: "MISO (SDO)"
- board text added: "MOSI (SDI)"
- board text added: "R"
- board text added: "RESET"
- board text added: "RX"
- board text added: "SCLK"
- board text added: "SD CS"
- board text added: "SD MISO"
- board text added: "SD MOSI"
- board text added: "SD SCK"
- board text added: "SW1"
- board text added: "SW2"
- board text added: "SW3"
- board text added: "SW4"
- board text added: "SW5"
- board text added: "SW6"
- board text added: "TX"
- board text added: "W"
