File: hardware/Deck_Mainboard/Deck_Mainboard.kicad_sch (KiCad schematic)
At the start: 58 parts, among them J1 LCD, J2 DEBUG, J3 SD, J4 BUTTONS, J5 Connector, USB-TYPE-C-16P, J6 ENCODERS, J7 ADDITIONAL PINS, SW1 BOOTSEL, SW2 RESET, U2 AP2112K-3.3, U3 W25Q128JVS, U4 USBLC6-2SC6, U5 APS6404L-3SQRx-SN, U6 RP2350B, X1 ABM8-272-T3

Commit message: hw: initial pcb layout
Parts:
- removed H1, H2, H3, H4: MH, symbol Mechanical:MountingHole_Pad
- removed J5: Connector, USB-TYPE-C-16P, PCM_JLCPCB:TYPE-C-SMD_HX-TYPE-C-16PIN, symbol PCM_JLCPCB-Extended:Connector, USB-TYPE-C-16P
- added H1, H2, H3, H4, H5, H6: MH, MountingHole:MountingHole_3.2mm_M3, symbol Mechanical:MountingHole
- added J8: USB_C_Receptacle_USB2.0_16P, deckLib:USB_C_4805, symbol Connector:USB_C_Receptacle_USB2.0_16P
- C1: renamed from C22; footprint (none) -> Capacitor_SMD:C_0402_1005Metric_Pad0.74x0.62mm_HandSolder
- C10: renamed from C13; footprint (none) -> Capacitor_SMD:C_0402_1005Metric_Pad0.74x0.62mm_HandSolder
- C11: renamed from C9; footprint (none) -> Capacitor_SMD:C_0402_1005Metric_Pad0.74x0.62mm_HandSolder
- C12: renamed from C14; footprint (none) -> Capacitor_SMD:C_0402_1005Metric_Pad0.74x0.62mm_HandSolder
- C13: renamed from C16; footprint (none) -> Capacitor_SMD:C_0402_1005Metric_Pad0.74x0.62mm_HandSolder
- C14: renamed from C10; footprint (none) -> Capacitor_SMD:C_0402_1005Metric_Pad0.74x0.62mm_HandSolder
- C15: renamed from C18; footprint (none) -> Capacitor_SMD:C_0402_1005Metric_Pad0.74x0.62mm_HandSolder
- C16: renamed from C19; footprint (none) -> Capacitor_SMD:C_0402_1005Metric_Pad0.74x0.62mm_HandSolder
- C17: renamed from C20; footprint (none) -> Capacitor_SMD:C_0402_1005Metric_Pad0.74x0.62mm_HandSolder
- C18: renamed from C21; footprint (none) -> Capacitor_SMD:C_0402_1005Metric_Pad0.74x0.62mm_HandSolder
- C19: renamed from C7; footprint (none) -> Capacitor_SMD:C_0402_1005Metric_Pad0.74x0.62mm_HandSolder
- C2: renamed from C23; footprint (none) -> Capacitor_SMD:C_0402_1005Metric_Pad0.74x0.62mm_HandSolder
- C20: renamed from C15; footprint (none) -> Capacitor_SMD:C_0402_1005Metric_Pad0.74x0.62mm_HandSolder
- C21: renamed from C8; footprint (none) -> Capacitor_SMD:C_0402_1005Metric_Pad0.74x0.62mm_HandSolder
- C3: renamed from C24; footprint (none) -> Capacitor_SMD:C_0402_1005Metric_Pad0.74x0.62mm_HandSolder
- C4: renamed from C5; value 1u -> 10u; footprint (none) -> Capacitor_SMD:C_0402_1005Metric_Pad0.74x0.62mm_HandSolder
- C5: renamed from C6; footprint (none) -> Capacitor_SMD:C_0402_1005Metric_Pad0.74x0.62mm_HandSolder
- C6: renamed from C1; footprint (none) -> Capacitor_SMD:C_0402_1005Metric_Pad0.74x0.62mm_HandSolder
- C7: renamed from C2; footprint (none) -> Capacitor_SMD:C_0402_1005Metric_Pad0.74x0.62mm_HandSolder
- C8: renamed from C3; footprint (none) -> Capacitor_SMD:C_0402_1005Metric_Pad0.74x0.62mm_HandSolder
- C9: renamed from C4; footprint (none) -> Capacitor_SMD:C_0402_1005Metric_Pad0.74x0.62mm_HandSolder
- D1: footprint (none) -> LED_SMD:LED_0603_1608Metric_Pad1.05x0.95mm_HandSolder
- J5: renamed from J3; footprint (none) -> Connector_PinHeader_2.54mm:PinHeader_1x04_P2.54mm_Vertical
- J6: renamed from J7; footprint (none) -> Connector_PinHeader_2.54mm:PinHeader_1x12_P2.54mm_Vertical
- R1: renamed from R16; footprint (none) -> Resistor_SMD:R_0402_1005Metric_Pad0.72x0.64mm_HandSolder
- R10: renamed from R8; footprint (none) -> Resistor_SMD:R_0402_1005Metric_Pad0.72x0.64mm_HandSolder
- R11: renamed from R6; footprint (none) -> Resistor_SMD:R_0402_1005Metric_Pad0.72x0.64mm_HandSolder
- R12: renamed from R18; footprint (none) -> Resistor_SMD:R_0402_1005Metric_Pad0.72x0.64mm_HandSolder
- R13: renamed from R14; footprint (none) -> Resistor_SMD:R_0402_1005Metric_Pad0.72x0.64mm_HandSolder
- R14: renamed from R10; footprint (none) -> Resistor_SMD:R_0402_1005Metric_Pad0.72x0.64mm_HandSolder
- R2: renamed from R12; footprint (none) -> Resistor_SMD:R_0402_1005Metric_Pad0.72x0.64mm_HandSolder
- R3: renamed from R13; footprint (none) -> Resistor_SMD:R_0402_1005Metric_Pad0.72x0.64mm_HandSolder
- R4: renamed from R1; footprint (none) -> Resistor_SMD:R_0402_1005Metric_Pad0.72x0.64mm_HandSolder
- R5: renamed from R2; footprint (none) -> Resistor_SMD:R_0402_1005Metric_Pad0.72x0.64mm_HandSolder
- R6: renamed from R5; footprint (none) -> Resistor_SMD:R_0402_1005Metric_Pad0.72x0.64mm_HandSolder
- R7: renamed from R15; footprint (none) -> Resistor_SMD:R_0402_1005Metric_Pad0.72x0.64mm_HandSolder
- R8: renamed from R11; footprint (none) -> Resistor_SMD:R_0402_1005Metric_Pad0.72x0.64mm_HandSolder
- R9: renamed from R17; footprint (none) -> Resistor_SMD:R_0402_1005Metric_Pad0.72x0.64mm_HandSolder
- SW1: value BOOTSEL -> RESET; footprint (none) -> Button_Switch_SMD:SW_Push_1P1T_NO_E-Switch_TL3301NxxxxxG
- SW2: value RESET -> BOOTSEL; footprint (none) -> Button_Switch_SMD:SW_Push_1P1T_NO_E-Switch_TL3301NxxxxxG
- renumbered J4 to J2, J6 to J3, J1 to J4, J2 to J7, U6 to U1, U4 to U2, U2 to U3, U5 to U4, U3 to U5
Connections:
- net GND: now also SW2.2, X1.4, J8.A1 (GND), J8.A12 (GND), J8.B1 (GND), J8.B12 (GND), J8.SH (SHIELD); no longer SW1.2, X1.3
- net RUN: now also SW1.1; no longer SW2.1
- net at R5.1: now also J8.B5 (CC2)
- net at R4.1: now also J8.A5 (CC1)
- net at R13.1: now also SW1.2; no longer SW2.2
- net at R12.2: now also SW2.1; no longer SW1.1
- net at F1.1: now also J8.A4 (VBUS), J8.A9 (VBUS), J8.B4 (VBUS), J8.B9 (VBUS)
- net USB_N: now reaches U2.1 (I/O1)
- net USB_N: now also J8.A7 (D-), J8.B7 (D-)
- net USB_P: now reaches U2.3 (I/O2)
- net USB_P: now also J8.A6 (D+), J8.B6 (D+)
- net at C21.1, R14.2: now also X1.3; no longer X1.4
Other:
- moved on the sheet: C21, R14

Commit message: temporary commit for validation
Connections:
- net SW1: now also J2.7 (Pin_7); no longer J2.2 (Pin_2)
- net SW2: now also J2.6 (Pin_6); no longer J2.3 (Pin_3)
- net SW3: now also J2.5 (Pin_5); no longer J2.4 (Pin_4)
- net SW4: now also J2.4 (Pin_4); no longer J2.5 (Pin_5)
- net SW5: now also J2.3 (Pin_3); no longer J2.6 (Pin_6)
- net SW6: now also J2.2 (Pin_2); no longer J2.7 (Pin_7)
Changed lines of the file:
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@@
 		)
 	)
-	(label "SW1"
+	(label "SW6"
 		(at 241.3 50.8 0)
 		(effects
@@
 		)
 	)
-	(label "SW6"
+	(label "SW1"
 		(at 241.3 63.5 0)
 		(effects
@@
 		)
 	)
-	(label "SW5"
+	(label "SW2"
 		(at 241.3 60.96 0)
 		(effects
@@
 		)
 	)
-	(label "SW2"
+	(label "SW5"
 		(at 241.3 53.34 0)
 		(effects
@@
 		)
 	)
-	(label "SW4"
+	(label "SW3"
 		(at 241.3 58.42 0)
 		(effects
@@
 		)
 	)
-	(label "SW3"
+	(label "SW4"
 		(at 241.3 55.88 0)
 		(effects

Commit message: hw: pcbs complete
Parts:
- removed H5, H6: MH, MountingHole:MountingHole_3.2mm_M3, symbol Mechanical:MountingHole
- added H5, H6: MH_P, MountingHole:MountingHole_3.2mm_M3_Pad, symbol Mechanical:MountingHole_Pad
- J8: footprint deckLib:USB_C_4805 -> deckLib:USB_C_vertical; TME https://www.tme.eu/pl/details/usb4805-03-a/zlacza-usb-i-iee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 -> https://www.tme.eu/pl/details/usb4145-03-0230-c/zlacza-usb-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
- X1: footprint Crystal:ABM8-272-T3_ABR -> deckLib:ABM8-272-T3_ABR
Connections:
- net +5V: now also C4.1, CR1.1, R6.2, U3.1 (VIN); no longer CR1.2, F1.2, U2.5 (VBUS)
- net GND: now also H5.1, H6.1
- new net VBUS: CR1.2, F1.2, U2.5 (VBUS)
Other:
- moved on the sheet: H1, H2, H3, H4
