File: hardware/Deck_ButtonBoard/ButtonBoard/ButtonBoard.kicad_pcb (KiCad board)
At the start: 2 copper layers, 98 x 62 mm, 29 parts, among them J1 Buttons, SW1_1 SW_Push, SW1_2 SW_Push, SW1_3 SW_Push, SW1_4 SW_Push, SW2_1 SW_Push, SW2_2 SW_Push, SW2_3 SW_Push, SW2_4 SW_Push, SW3_1 SW_Push, SW3_2 SW_Push, SW3_3 SW_Push, SW3_4 SW_Push, SW4_1 SW_Push, SW4_2 SW_Push, SW4_3 SW_Push, SW4_4 SW_Push, SW5_1 SW_Push, SW5_2 SW_Push, SW5_3 SW_Push, SW5_4 SW_Push, SW6_1 SW_Push, SW6_2 SW_Push, SW6_3 SW_Push, SW6_4 SW_Push

Commit message: hw: pcbs complete
Connections:
- J1 pad 2: /SW6 -> /SW1
- J1 pad 3: /SW5 -> /SW2
- J1 pad 4: /SW4 -> /SW3
- J1 pad 5: /SW3 -> /SW4
- J1 pad 6: /SW2 -> /SW5
- J1 pad 7: /SW1 -> /SW6
- SW1_1 pad 1: /SW1 -> /SW6
- SW1_2 pad 1: /SW1 -> /SW6
- SW1_3 pad 1: /SW1 -> /SW6
- SW1_4 pad 1: /SW1 -> /SW6
- SW2_1 pad 1: /SW2 -> /SW5
- SW2_2 pad 1: /SW2 -> /SW5
- SW2_3 pad 1: /SW2 -> /SW5
- SW2_4 pad 1: /SW2 -> /SW5
- SW3_1 pad 1: /SW3 -> /SW4
- SW3_2 pad 1: /SW3 -> /SW4
- SW3_3 pad 1: /SW3 -> /SW4
- SW3_4 pad 1: /SW3 -> /SW4
- SW4_1 pad 1: /SW4 -> /SW3
- SW4_2 pad 1: /SW4 -> /SW3
- SW4_3 pad 1: /SW4 -> /SW3
- SW4_4 pad 1: /SW4 -> /SW3
- SW5_1 pad 1: /SW5 -> /SW2
- SW5_2 pad 1: /SW5 -> /SW2
- SW5_3 pad 1: /SW5 -> /SW2
- SW5_4 pad 1: /SW5 -> /SW2
- SW6_1 pad 1: /SW6 -> /SW1
- SW6_2 pad 1: /SW6 -> /SW1
- SW6_3 pad 1: /SW6 -> /SW1
- SW6_4 pad 1: /SW6 -> /SW1
Routing:
- net /SW2: track 139.2 -> 56.0 mm
- net /SW5: track 58.0 -> 139.9 mm, vias 3 -> 4
- net /SW6: track 85.9 -> 147.3 mm, vias 2 -> 0
- net /SW1: track 147.3 -> 85.9 mm, vias 0 -> 2
- net /SW3: track 114.8 -> 77.4 mm, vias 0 -> 4
- net /SW4: track 78.2 -> 114.8 mm, vias 4 -> 0
- net GND: track 1.74 -> 35.1 mm, vias 63 -> 89
Other:
- board text added: "2"
- board text added: "GND"
- board text added: "R"
- board text added: "SW1"
- board text added: "SW2"
- board text added: "SW3"
- board text added: "SW4"
- board text added: "SW5"
- board text added: "SW6"
- board text added: "W"
