File: hardware/Deck_ButtonBoard/ButtonBoard/ButtonBoard.kicad_sch (KiCad schematic)
At the start: 25 parts, among them J1 Buttons, SW1_1 SW_Push, SW1_2 SW_Push, SW1_3 SW_Push, SW1_4 SW_Push, SW2_1 SW_Push, SW2_2 SW_Push, SW2_3 SW_Push, SW2_4 SW_Push, SW3_1 SW_Push, SW3_2 SW_Push, SW3_3 SW_Push, SW3_4 SW_Push, SW4_1 SW_Push, SW4_2 SW_Push, SW4_3 SW_Push, SW4_4 SW_Push, SW5_1 SW_Push, SW5_2 SW_Push, SW5_3 SW_Push, SW5_4 SW_Push, SW6_1 SW_Push, SW6_2 SW_Push, SW6_3 SW_Push, SW6_4 SW_Push

Commit message: hw: pcbs complete
Connections:
- net SW1: now also J1.2 (Pin_2), SW6_1.1, SW6_2.1, SW6_3.1, SW6_4.1; no longer J1.7 (Pin_7), SW1_1.1, SW1_2.1, SW1_3.1, SW1_4.1
- net SW2: now also J1.3 (Pin_3), SW5_1.1, SW5_2.1, SW5_3.1, SW5_4.1; no longer J1.6 (Pin_6), SW2_1.1, SW2_2.1, SW2_3.1, SW2_4.1
- net SW3: now also J1.4 (Pin_4), SW4_1.1, SW4_2.1, SW4_3.1, SW4_4.1; no longer J1.5 (Pin_5), SW3_1.1, SW3_2.1, SW3_3.1, SW3_4.1
- net SW4: now also J1.5 (Pin_5), SW3_1.1, SW3_2.1, SW3_3.1, SW3_4.1; no longer J1.4 (Pin_4), SW4_1.1, SW4_2.1, SW4_3.1, SW4_4.1
- net SW5: now also J1.6 (Pin_6), SW2_1.1, SW2_2.1, SW2_3.1, SW2_4.1; no longer J1.3 (Pin_3), SW5_1.1, SW5_2.1, SW5_3.1, SW5_4.1
- net SW6: now also J1.7 (Pin_7), SW1_1.1, SW1_2.1, SW1_3.1, SW1_4.1; no longer J1.2 (Pin_2), SW6_1.1, SW6_2.1, SW6_3.1, SW6_4.1
Changed lines of the file:
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@@
 		)
 	)
-	(label "SW5"
+	(label "SW3"
+		(at 167.64 73.66 90)
+		(effects
+			(font
+				(size 1.27 1.27)
+			)
+			(justify left bottom)
+		)
+	)
+	(label "SW1"
+		(at 215.9 67.31 0)
+		(effects
+			(font
+				(size 1.27 1.27)
+			)
+			(justify left bottom)
+		)
+	)
+	(label "SW4"
+		(at 215.9 74.93 0)
+		(effects
+			(font
+				(size 1.27 1.27)
+			)
+			(justify left bottom)
+		)
+	)
+	(label "SW1"
+		(at 198.12 73.66 90)
+		(effects
+			(font
+				(size 1.27 1.27)
+			)
+			(justify left bottom)
+		)
+	)
+	(label "SW2"
 		(at 215.9 69.85 0)
 		(effects
@@
 		)
 	)
-	(label "SW3"
-		(at 215.9 74.93 0)
+	(label "SW4"
+		(at 152.4 73.66 90)
 		(effects
 			(font
@@
 		)
 	)
-	(label "SW6"
-		(at 198.12 73.66 90)
-		(effects
-			(font
-				(size 1.27 1.27)
-			)
-			(justify left bottom)
-		)
-	)
-	(label "SW4"
-		(at 215.9 72.39 0)
-		(effects
-			(font
-				(size 1.27 1.27)
-			)
-			(justify left bottom)
-		)
-	)
-	(label "SW2"
+	(label "SW5"
 		(at 215.9 77.47 0)
 		(effects
@@
 		)
 	)
-	(label "SW2"
-		(at 137.16 73.66 90)
+	(label "SW6"
+		(at 215.9 80.01 0)
 		(effects
 			(font
@@
 		)
 	)
-	(label "SW5"
+	(label "SW3"
+		(at 215.9 72.39 0)
+		(effects
+			(font
+				(size 1.27 1.27)
+			)
+			(justify left bottom)
+		)
+	)
+	(label "SW2"
 		(at 182.88 73.66 90)
 		(effects
@@
 		)
 	)
-	(label "SW3"
-		(at 152.4 73.66 90)
-		(effects
-			(font
-				(size 1.27 1.27)
-			)
-			(justify left bottom)
-		)
-	)
-	(label "SW4"
-		(at 167.64 73.66 90)
-		(effects
-			(font
-				(size 1.27 1.27)
-			)
-			(justify left bottom)
-		)
-	)
-	(label "SW1"
-		(at 215.9 80.01 0)
-		(effects
-			(font
-				(size 1.27 1.27)
-			)
-			(justify left bottom)
-		)
-	)
-	(label "SW1"
+	(label "SW6"
 		(at 121.92 73.66 90)
-		(effects
-			(font
-				(size 1.27 1.27)
-			)
-			(justify left bottom)
-		)
-	)
-	(label "SW6"
-		(at 215.9 67.31 0)
 		(effects
 			(font
@@
 		(effects
 			(font
+				(size 1.27 1.27)
+			)
+			(justify left bottom)
+		)
+	)
+	(label "SW5"
+		(at 137.16 73.66 90)
+		(effects
+			(font
